Commit message: positioning for cybertruck

File: submissions/2_go_chase_it/my_robot/urdf/my_robot.xacro (robot description, xacro)
@@ -22,5 +22,5 @@
       <origin xyz="0 0 0" rpy=" 0 0 0"/>
       <geometry>
-        <box size=".6 .2 .025"/>
+        <box size=".5 .2 .01"/>
       </geometry>
     </collision>
@@ -28,9 +28,11 @@
       <origin xyz="0 0 0" rpy=" 0 0 0"/>
       <geometry>
-        <box size=".55 .2 .025"/>
-      </geometry>
-    </visual>
+        <box size=".5 .2 .01"/>
+      </geometry>
+    </visual>
+    <!-- casters -->
+    <xacro:property name="caster_x" value="0.0" />
     <collision name='back_caster_collision'>
-      <origin xyz="0.2 -0.08 -0.03" rpy=" 0 0 0"/>
+      <origin xyz="${caster_x} -0.0 -0.03" rpy=" 0 0 0"/>
       <geometry>
         <sphere radius="0.0199"/>
@@ -38,26 +40,27 @@
     </collision>
     <visual name='back_caster_visual'>
-      <origin xyz="0.2 -0.08 -0.03" rpy=" 0 0 0"/>
+      <origin xyz="${caster_x} -0.0 -0.03" rpy=" 0 0 0"/>
       <geometry>
         <sphere radius="0.02"/>
       </geometry>
     </visual>
-    <collision name='front_caster_collision'>
-      <origin xyz="0.2 0.08 -0.03" rpy=" 0 0 0"/>
-      <geometry>
-        <sphere radius="0.0199"/>
-      </geometry>
-    </collision>
-    <visual name='front_caster_visual'>
-      <origin xyz="0.2 0.08 -0.03" rpy=" 0 0 0"/>
-      <geometry>
-        <sphere radius="0.02"/>
-      </geometry>
-    </visual>
-  </link>
-  <!-- Add back wheels -->
+    <!-- Add the Cybertruck -->
+    <visual>
+      <origin xyz="0.02 0 -0.05" rpy="0 0 0" />
+      <geometry>
+        <mesh filename="package://my_robot/meshes/cybertruck.stl"/>
+      </geometry>
+    </visual>
+    <collision>
+      <origin xyz="0 0 0" rpy="0 0 0" />
+      <geometry>
+        <box size=".5 .2 .01"/>
+      </geometry>
+    </collision>
+  </link>
+  <!-- Add wheels -->
   <xacro:property name="wheel_radius" value="0.04" />
   <xacro:property name="wheel_mass" value="10" />
-  <xacro:property name="wheel_inertia" value="0.1" />
+  <xacro:property name="wheel_inertia" value="0.2" />
   <link name='left_wheel'>
     <visual>
@@ -213,5 +216,5 @@
   </link>
   <joint type="fixed" name="camera_joint">
-    <origin xyz=".2 0 0" rpy="0 0 0"/>
+    <origin xyz=".25 0 .03" rpy="0 0 0"/>
     <child link="camera"/>
     <parent link="chassis"/>
@@ -242,5 +245,5 @@
   </link>
   <joint type="fixed" name="hokuyo_joint">
-    <origin xyz=".15 0 .1" rpy="0 0 0"/>
+    <origin xyz=".0 0 .125" rpy="0 0 0"/>
     <child link="hokuyo"/>
     <parent link="chassis"/>
@@ -249,44 +252,14 @@
   <!-- Add colors -->
   <gazebo reference="left_wheel">
-    <material>Gazebo/Green</material>
+    <material>Gazebo/Black</material>
   </gazebo>
   <gazebo reference="right_wheel">
-    <material>Gazebo/Green</material>
+    <material>Gazebo/Black</material>
   </gazebo>
   <gazebo reference="chassis">
-    <material>Gazebo/Blue</material>
+    <material>Gazebo/Gray</material>
   </gazebo>
   <gazebo reference="camera">
-    <material>Gazebo/Red</material>
-  </gazebo>
-  <!-- Add Cybertruck -->
-  <link name="cybertruck">
-    <visual>
-      <origin xyz="0 0 0" rpy="0 0 0" />
-      <geometry>
-        <mesh filename="package://my_robot/meshes/cybertruck.stl"/>
-      </geometry>
-    </visual>
-    <collision>
-      <origin xyz="0 0 0" rpy="0 0 0" />
-      <geometry>
-        <box size=".01 .01 .01"/>
-      </geometry>
-    </collision>
-    <inertial>
-      <mass value="1e-5"/>
-      <origin xyz="0 0 0" rpy=" 0 0 0"/>
-      <inertia
-        ixx="1e-6" ixy="0" ixz="0"
-        iyy="1e-6" iyz="0"
-        izz="1e-6"
-      />
-    </inertial>
-  </link>
-  <joint type="fixed" name="cybertruck_joint">
-    <origin xyz="0 0 0" rpy="0 0 0"/>
-    <child link="cybertruck"/>
-    <parent link="chassis"/>
-    <axis xyz="0 1 0" rpy="0 0 0"/>
-  </joint>
+    <material>Gazebo/Black</material>
+  </gazebo>
 </robot>

Commit message: fix: wheels and caster position for better rotation ability

File: submissions/2_go_chase_it/my_robot/urdf/my_robot.xacro (robot description, xacro)
@@ -11,10 +11,10 @@
     <pose>0 0 0.0525 0 0 0</pose>
     <inertial>
-      <mass value="3.0"/>
-      <origin xyz="0 0 0" rpy=" 0 0 0"/>
-      <inertia
-          ixx="0.02" ixy="0" ixz="0"
-          iyy="0.02" iyz="0"
-          izz="0.02"
+      <mass value="10.0"/>
+      <origin xyz="0 0 0" rpy=" 0 0 0"/>
+      <inertia
+          ixx="0.1" ixy="0" ixz="0"
+          iyy="0.1" iyz="0"
+          izz="0.1"
       />
     </inertial>
@@ -32,5 +32,5 @@
     </visual>
     <!-- casters -->
-    <xacro:property name="caster_x" value="0.0" />
+    <xacro:property name="caster_x" value="0.1" />
     <collision name='back_caster_collision'>
       <origin xyz="${caster_x} -0.0 -0.03" rpy=" 0 0 0"/>
@@ -41,4 +41,16 @@
     <visual name='back_caster_visual'>
       <origin xyz="${caster_x} -0.0 -0.03" rpy=" 0 0 0"/>
+      <geometry>
+        <sphere radius="0.02"/>
+      </geometry>
+    </visual>
+    <collision name='front_caster_collision'>
+      <origin xyz="-${caster_x} -0.0 -0.03" rpy=" 0 0 0"/>
+      <geometry>
+        <sphere radius="0.0199"/>
+      </geometry>
+    </collision>
+    <visual name='front_caster_visual'>
+      <origin xyz="-${caster_x} -0.0 -0.03" rpy=" 0 0 0"/>
       <geometry>
         <sphere radius="0.02"/>
@@ -87,5 +99,5 @@
   </link>
   <joint type="continuous" name="left_wheel_hinge">
-    <origin xyz="-.18 0.083 -0.01" rpy="0 0 0"/>
+    <origin xyz="0 0.083 -0.01" rpy="0 0 0"/>
     <child link="left_wheel"/>
     <parent link="chassis"/>
@@ -118,5 +130,5 @@
   </link>
   <joint type="continuous" name="right_wheel_hinge">
-    <origin xyz="-.18 -0.083 -0.01" rpy="0 0 0"/>
+    <origin xyz="0 -0.083 -0.01" rpy="0 0 0"/>
     <child link="right_wheel"/>
     <parent link="chassis"/>
@@ -252,8 +264,8 @@
   <!-- Add colors -->
   <gazebo reference="left_wheel">
-    <material>Gazebo/Black</material>
+    <material>Gazebo/Grey</material>
   </gazebo>
   <gazebo reference="right_wheel">
-    <material>Gazebo/Black</material>
+    <material>Gazebo/Grey</material>
   </gazebo>
   <gazebo reference="chassis">
